File: Isolated_Signal_Transfer_0.2/Isolated_Signal_Transfer_0.2.sch (KiCad schematic (older format))
At the start: 23 parts, among them J1 Conn_01x02_Male, J2 Conn_01x02_Male, J3 Conn_01x02_Male, J4 Conn_01x02_Male, U1 LM358, U2 IL300, U3 LM358

Commit message: Changes
Parts:
- removed J3, J4: Conn_01x02_Male, Connector_PinHeader_2.54mm:PinHeader_1x02_P2.54mm_Vertical, symbol Connector:Conn_01x02_Male
- added D3: YELLOW, LED_SMD:LED_0805_2012Metric, symbol Device:LED
- added D4: RED, LED_SMD:LED_0805_2012Metric, symbol Device:LED
- added J3: Conn_01x04, Connector_PinHeader_2.54mm:PinHeader_1x04_P2.54mm_Vertical, symbol Connector_Generic:Conn_01x04
- added R10: 50K, Resistor_SMD:R_0603_1608Metric, symbol Device:R
- added R11, R14, R15: 1K, Resistor_SMD:R_0603_1608Metric, symbol Device:R
- added R13: 100K, Resistor_SMD:R_0603_1608Metric, symbol Device:R
- renumbered R10 to R12
Connections:
- net +24V: now also D4.2 (A), J3.1 (Pin_1), R10.1, R14.1; no longer U3.5 (+)
- net GND: now also J3.3 (Pin_3), J3.4 (Pin_4), R11.2, R15.2; no longer U3.6 (-)
- net at R12.1, U3.1: now also U3.6 (-), J3.2 (Pin_2)
- net at U3.7: now also D3.1 (K), R13.2
- new net: R10.2, R11.1, R13.1, U3.5 (+)
- new net: D4.1 (K), R15.1
- new net: D3.2 (A), R14.2
Other:
- note added: "HV indicator\n>60 V!"
- note added: "Power Indicator"
- moved on the sheet: U3B
Changed lines of the file:
@@
 EESchema Schematic File Version 4
-LIBS:Isolated_Signal_Transfer_0.1-cache
+LIBS:Isolated_Signal_Transfer_0.2-cache
 EELAYER 30 0
 EELAYER END
@@
 	1400 2800 1400 2900
 $Comp
+L Connector_Generic:Conn_01x04 J3
+U 1 1 5D77E214
+P 8900 3500
+F 0 "J3" H 8980 3492 50  0000 L CNN
+F 1 "Conn_01x04" H 8980 3401 50  0000 L CNN
+F 2 "Connector_PinHeader_2.54mm:PinHeader_1x04_P2.54mm_Vertical" H 8900 3500 50  0001 C CNN
+F 3 "~" H 8900 3500 50  0001 C CNN
+	1    8900 3500
+	1    0    0    -1
+$EndComp
+$Comp
 L power:+24V #PWR020
 U 1 1 5D77F59D
@@
 L power:GND #PWR021
 U 1 1 5D77FF2B
-P 8700 3850
-F 0 "#PWR021" H 8700 3600 50  0001 C CNN
-F 1 "GND" H 8705 3677 50  0000 C CNN
-F 2 "" H 8700 3850 50  0001 C CNN
-F 3 "" H 8700 3850 50  0001 C CNN
-	1    8700 3850
+P 8700 3700
+F 0 "#PWR021" H 8700 3450 50  0001 C CNN
+F 1 "GND" H 8705 3527 50  0000 C CNN
+F 2 "" H 8700 3700 50  0001 C CNN
+F 3 "" H 8700 3700 50  0001 C CNN
+	1    8700 3700
 	1    0    0    -1
 $EndComp
@@
 Connection ~ 2950 2900
 Wire Wire Line
-	8700 3750 8700 3850
+	8700 3600 8700 3700
+Connection ~ 8700 3700
 Connection ~ 5900 3200
 Wire Wire Line
@@
 Connection ~ 7450 3500
 $Comp
-L Device:R R10
+L Device:R R12
 U 1 1 5D6E30BA
 P 7750 3500
-F 0 "R10" H 7820 3546 50  0000 L CNN
+F 0 "R12" H 7820 3546 50  0000 L CNN
 F 1 "5K" H 7820 3455 50  0000 L CNN
 F 2 "Resistor_SMD:R_0603_1608Metric" V 7680 3500 50  0001 C CNN
@@
 L Amplifier_Operational:LM358 U3
 U 2 1 5D6FFD52
-P 7850 1350
-F 0 "U3" H 7850 1717 50  0000 C CNN
-F 1 "LM358" H 7850 1626 50  0000 C CNN
-F 2 "Package_SO:SOIC-8_3.9x4.9mm_P1.27mm" H 7850 1350 50  0001 C CNN
-F 3 "http://www.ti.com/lit/ds/symlink/lm2904-n.pdf" H 7850 1350 50  0001 C CNN
-	2    7850 1350
-	1    0    0    -1
-$EndComp
-$Comp
-L power:GND #PWR017
-U 1 1 5D706A90
-P 7550 1450
-F 0 "#PWR017" H 7550 1200 50  0001 C CNN
-F 1 "GND" H 7555 1277 50  0000 C CNN
-F 2 "" H 7550 1450 50  0001 C CNN
-F 3 "" H 7550 1450 50  0001 C CNN
-	1    7550 1450
+P 8100 2200
+F 0 "U3" H 8100 2567 50  0000 C CNN
+F 1 "LM358" H 8100 2476 50  0000 C CNN
+F 2 "Package_SO:SOIC-8_3.9x4.9mm_P1.27mm" H 8100 2200 50  0001 C CNN
+F 3 "http://www.ti.com/lit/ds/symlink/lm2904-n.pdf" H 8100 2200 50  0001 C CNN
+	2    8100 2200
 	1    0    0    -1
 $EndComp
@@
 L power:+24V #PWR016
 U 1 1 5D7072C0
-P 7550 1250
-F 0 "#PWR016" H 7550 1100 50  0001 C CNN
-F 1 "+24V" H 7565 1423 50  0000 C CNN
-F 2 "" H 7550 1250 50  0001 C CNN
-F 3 "" H 7550 1250 50  0001 C CNN
-	1    7550 1250
-	1    0    0    -1
-$EndComp
-$Comp
-L Connector:Conn_01x02_Male J3
-U 1 1 5D738A78
-P 8900 3500
-F 0 "J3" H 8872 3382 50  0000 R CNN
-F 1 "Conn_01x02_Male" H 8872 3473 50  0000 R CNN
-F 2 "Connector_PinHeader_2.54mm:PinHeader_1x02_P2.54mm_Vertical" H 8900 3500 50  0001 C CNN
-F 3 "~" H 8900 3500 50  0001 C CNN
-	1    8900 3500
-	-1   0    0    1
-$EndComp
-$Comp
-L Connector:Conn_01x02_Male J4
-U 1 1 5D73A3AA
-P 8900 3850
-F 0 "J4" H 8872 3732 50  0000 R CNN
-F 1 "Conn_01x02_Male" H 8872 3823 50  0000 R CNN
-F 2 "Connector_PinHeader_2.54mm:PinHeader_1x02_P2.54mm_Vertical" H 8900 3850 50  0001 C CNN
-F 3 "~" H 8900 3850 50  0001 C CNN
-	1    8900 3850
-	-1   0    0    1
-$EndComp
-Connection ~ 8700 3850
+P 7500 1800
+F 0 "#PWR016" H 7500 1650 50  0001 C CNN
+F 1 "+24V" H 7515 1973 50  0000 C CNN
+F 2 "" H 7500 1800 50  0001 C CNN
+F 3 "" H 7500 1800 50  0001 C CNN
+	1    7500 1800
+	1    0    0    -1
+$EndComp
+$Comp
+L Device:LED D4
+U 1 1 5D737E47
+P 9500 1150
+F 0 "D4" V 9539 1032 50  0000 R CNN
+F 1 "RED" V 9448 1032 50  0000 R CNN
+F 2 "LED_SMD:LED_0805_2012Metric" H 9500 1150 50  0001 C CNN
+F 3 "~" H 9500 1150 50  0001 C CNN
+	1    9500 1150
+	0    -1   -1   0
+$EndComp
+$Comp
+L Device:LED D3
+U 1 1 5D739BD3
+P 8850 2200
+F 0 "D3" H 8843 2416 50  0000 C CNN
+F 1 "YELLOW" H 8843 2325 50  0000 C CNN
+F 2 "LED_SMD:LED_0805_2012Metric" H 8850 2200 50  0001 C CNN
+F 3 "~" H 8850 2200 50  0001 C CNN
+	1    8850 2200
+	1    0    0    -1
+$EndComp
+$Comp
+L power:+24V #PWR023
+U 1 1 5D73B9C5
+P 9500 1000
+F 0 "#PWR023" H 9500 850 50  0001 C CNN
+F 1 "+24V" H 9515 1173 50  0000 C CNN
+F 2 "" H 9500 1000 50  0001 C CNN
+F 3 "" H 9500 1000 50  0001 C CNN
+	1    9500 1000
+	1    0    0    -1
+$EndComp
+$Comp
+L power:GND #PWR024
+U 1 1 5D73C3E0
+P 9500 1600
+F 0 "#PWR024" H 9500 1350 50  0001 C CNN
+F 1 "GND" H 9505 1427 50  0000 C CNN
+F 2 "" H 9500 1600 50  0001 C CNN
+F 3 "" H 9500 1600 50  0001 C CNN
+	1    9500 1600
+	1    0    0    -1
+$EndComp
+$Comp
+L Device:R R15
+U 1 1 5D73CDB0
+P 9500 1450
+F 0 "R15" H 9570 1496 50  0000 L CNN
+F 1 "1K" H 9570 1405 50  0000 L CNN
+F 2 "Resistor_SMD:R_0603_1608Metric" V 9430 1450 50  0001 C CNN
+F 3 "~" H 9500 1450 50  0001 C CNN
+	1    9500 1450
+	1    0    0    -1
+$EndComp
+$Comp
+L power:+24V #PWR022
+U 1 1 5D745A5F
+P 9200 1900
+F 0 "#PWR022" H 9200 1750 50  0001 C CNN
+F 1 "+24V" H 9215 2073 50  0000 C CNN
+F 2 "" H 9200 1900 50  0001 C CNN
+F 3 "" H 9200 1900 50  0001 C CNN
+	1    9200 1900
+	1    0    0    -1
+$EndComp
+$Comp
+L Device:R R14
+U 1 1 5D746D5E
+P 9200 2050
+F 0 "R14" H 9270 2096 50  0000 L CNN
+F 1 "1K" H 9270 2005 50  0000 L CNN
+F 2 "Resistor_SMD:R_0603_1608Metric" V 9130 2050 50  0001 C CNN
+F 3 "~" H 9200 2050 50  0001 C CNN
+	1    9200 2050
+	1    0    0    -1
+$EndComp
+Wire Wire Line
+	9200 2200 9000 2200
+Wire Wire Line
+	8700 2200 8450 2200
+$Comp
+L Device:R R10
+U 1 1 5D74C52C
+P 7500 1950
+F 0 "R10" H 7570 1996 50  0000 L CNN
+F 1 "50K" H 7570 1905 50  0000 L CNN
+F 2 "Resistor_SMD:R_0603_1608Metric" V 7430 1950 50  0001 C CNN
+F 3 "~" H 7500 1950 50  0001 C CNN
+	1    7500 1950
+	1    0    0    -1
+$EndComp
+$Comp
+L Device:R R11
+U 1 1 5D74CB21
+P 7500 2250
+F 0 "R11" H 7570 2296 50  0000 L CNN
+F 1 "1K" H 7570 2205 50  0000 L CNN
+F 2 "Resistor_SMD:R_0603_1608Metric" V 7430 2250 50  0001 C CNN
+F 3 "~" H 7500 2250 50  0001 C CNN
+	1    7500 2250
+	1    0    0    -1
+$EndComp
+$Comp
+L power:GND #PWR017
+U 1 1 5D74CD93
+P 7500 2400
+F 0 "#PWR017" H 7500 2150 50  0001 C CNN
+F 1 "GND" H 7505 2227 50  0000 C CNN
+F 2 "" H 7500 2400 50  0001 C CNN
+F 3 "" H 7500 2400 50  0001 C CNN
+	1    7500 2400
+	1    0    0    -1
+$EndComp
+Connection ~ 7500 2100
+Wire Wire Line
+	7800 2300 7800 2700
+Wire Wire Line
+	7800 2700 8050 2700
+Wire Wire Line
+	8050 2700 8050 3200
+Connection ~ 8050 3200
+Text Notes 8600 2450 0    50   ~ 0
+HV indicator\n>60 V!
+$Comp
+L Device:R R13
+U 1 1 5D75121A
+P 8450 2050
+F 0 "R13" H 8520 2096 50  0000 L CNN
+F 1 "100K" H 8520 2005 50  0000 L CNN
+F 2 "Resistor_SMD:R_0603_1608Metric" V 8380 2050 50  0001 C CNN
+F 3 "~" H 8450 2050 50  0001 C CNN
+	1    8450 2050
+	1    0    0    -1
+$EndComp
+Connection ~ 8450 2200
+Wire Wire Line
+	8450 2200 8400 2200
+Wire Wire Line
+	8450 1900 7800 1900
+Wire Wire Line
+	7800 1900 7800 2100
+Wire Wire Line
+	7500 2100 7800 2100
+Connection ~ 7800 2100
+Text Notes 9200 1050 0    50   ~ 0
+Power Indicator
 $EndSCHEMATC
